Commit message: Add l515 link

File: nextage_tutorials/urdf/JSKNextageOpen.urdf (robot description, URDF)
Before this commit: robot NextageOpen, 17 links, 16 joints
Links:
- added link l515_head_link
Joints:
- added joint l515_head_JOINT: type fixed, parent HEAD_JOINT1_Link, child l515_head_link, origin xyz=0 0 0.08 rpy=3.14 -1.57 0
