Commit message: Add JSKNextageOpen.urdf and jsk-nextage.l

File: nextage_tutorials/urdf/JSKNextageOpen.urdf (robot description, URDF)
Before this commit: robot NextageOpen, 21 links, 20 joints
Links:
- removed link ftsensor_l_link
- removed link ftsensor_r_link
- removed link l515_head_link
- removed link nextage_to_ftsensor_l_link
- removed link nextage_to_ftsensor_r_link
- added link CHEST_L515_Link; collision mesh filename=package://nextage_tutorials/meshes/CHEST_L515.stl scale=0.001 0.001 0.001; visual mesh filename=package://nextage_tutorials/meshes/CHEST_L515.stl scale=0.001 0.001 0.001
- added link CHEST_NEXTAGE_TO_L515_Link; collision mesh filename=package://nextage_tutorials/meshes/CHEST_NEXTAGE_TO_L515.stl scale=0.001 0.001 0.001; visual mesh filename=package://nextage_tutorials/meshes/CHEST_NEXTAGE_TO_L515.stl scale=0.001 0.001 0.001
- added link L515_Link; collision mesh filename=package://nextage_tutorials/meshes/L515.stl scale=0.001 0.001 0.001; visual mesh filename=package://nextage_tutorials/meshes/L515.stl scale=0.001 0.001 0.001
- added link LARM_FTSENSOR_Link; collision mesh filename=package://nextage_tutorials/meshes/LARM_FTSENSOR.stl scale=0.001 0.001 0.001; visual mesh filename=package://nextage_tutorials/meshes/LARM_FTSENSOR.stl scale=0.001 0.001 0.001
- added link LARM_FTSENSOR_SPACER_Link; collision cylinder length=0.0175 radius=0.0185; visual cylinder length=0.0175 radius=0.0185
- added link LARM_NEJINEJI_Link; collision mesh filename=package://nextage_tutorials/meshes/LARM_NEJINEJI.stl scale=0.001 0.001 0.001; visual mesh filename=package://nextage_tutorials/meshes/LARM_NEJINEJI.stl scale=0.001 0.001 0.001
- added link LARM_NEXTAGE_TO_FTSENSOR_Link; collision mesh filename=package://nextage_tutorials/meshes/LARM_NEXTAGE_TO_FTSENSOR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 scale=0.001 0.001 0.001; visual mesh filename=package://nextage_tutorials/meshes/LARM_NEXTAGE_TO_FTSENSOR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 scale=0.001 0.001 0.001
- added link RARM_FTSENSOR_Link; collision mesh filename=package://nextage_tutorials/meshes/RARM_FTSENSOR.stl scale=0.001 0.001 0.001; visual mesh filename=package://nextage_tutorials/meshes/RARM_FTSENSOR.stl scale=0.001 0.001 0.001
- added link RARM_FTSENSOR_SPACER_Link; collision cylinder length=0.0175 radius=0.0185; visual cylinder length=0.0175 radius=0.0185
- added link RARM_NEJINEJI_Link; collision mesh filename=package://nextage_tutorials/meshes/RARM_NEJINEJI.stl scale=0.001 0.001 0.001; visual mesh filename=package://nextage_tutorials/meshes/RARM_NEJINEJI.stl scale=0.001 0.001 0.001
- added link RARM_NEXTAGE_TO_FTSENSOR_Link; collision mesh filename=package://nextage_tutorials/meshes/RARM_NEXTAGE_TO_FTSENSOR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 scale=0.001 0.001 0.001; visual mesh filename=package://nextage_tutorials/meshes/RARM_NEXTAGE_TO_FTSENSOR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 scale=0.001 0.001 0.001
- link LARM_JOINT5_Link: geometry 
- link RARM_JOINT5_Link: geometry 
Joints:
- removed joint LARM_JOINT5_to_nextage_to_ftsensor_l
- removed joint RARM_JOINT5_to_nextage_to_ftsensor_r
- removed joint l515_head_JOINT
- removed joint nextage_to_ftsensor_l_to_ftsensor_l
- removed joint nextage_to_ftsensor_r_to_ftsensor_r
- added joint CHEST_JOINT0_TO_NEXTAGE_TO_L515: type fixed, parent CHEST_JOINT0_Link, child CHEST_NEXTAGE_TO_L515_Link, origin xyz=0.080855 0.099197 0.291294 rpy=0.698132 0 -1.570796
- added joint CHEST_L515_TO_L515: type fixed, parent CHEST_L515_Link, child L515_Link, origin xyz=0 0 0 rpy=0 0 0
- added joint CHEST_NEXTAGE_TO_L515_TO_CHEST_L515: type fixed, parent CHEST_NEXTAGE_TO_L515_Link, child CHEST_L515_Link, origin xyz=0.099197 0.069502 0.025 rpy=-1.570796 1.570796 0
- added joint LARM_FTSENSOR_SPACER_TO_NEXTAGE_TO_FTSENSOR: type fixed, parent LARM_FTSENSOR_SPACER_Link, child LARM_NEXTAGE_TO_FTSENSOR_Link, origin xyz=-0.0165 -0.0275 0.0275 rpy=0 1.570796 0
- added joint LARM_FTSENSOR_TO_NEJINEJI: type fixed, parent LARM_FTSENSOR_Link, child LARM_NEJINEJI_Link, origin xyz=-0.03634 0.03631 -0.01197 rpy=-1.570796 0 -1.570796
- added joint LARM_JOINT5_TO_FTSENSOR_SPACER: type fixed, parent LARM_JOINT5_Link, child LARM_FTSENSOR_SPACER_Link, origin xyz=0.015 0 0 rpy=0 0 0
- added joint LARM_NEXTAGE_TO_FTSENSOR_TO_FTSENSOR: type fixed, parent LARM_NEXTAGE_TO_FTSENSOR_Link, child LARM_FTSENSOR_Link, origin xyz=0.0275 0.0275 -0.017 rpy=0 0 -0.785398
- added joint RARM_FTSENSOR_SPACER_TO_NEXTAGE_TO_FTSENSOR: type fixed, parent RARM_FTSENSOR_SPACER_Link, child RARM_NEXTAGE_TO_FTSENSOR_Link, origin xyz=-0.0165 -0.0275 0.0275 rpy=0 1.570796 0
- added joint RARM_FTSENSOR_TO_NEJINEJI: type fixed, parent RARM_FTSENSOR_Link, child RARM_NEJINEJI_Link, origin xyz=0.03634 -0.03631 -0.01197 rpy=-1.570796 0 1.570796
- added joint RARM_JOINT5_TO_FTSENSOR_SPACER: type fixed, parent RARM_JOINT5_Link, child RARM_FTSENSOR_SPACER_Link, origin xyz=0.015 0 0 rpy=0 0 0
- added joint RARM_NEXTAGE_TO_FTSENSOR_TO_FTSENSOR: type fixed, parent RARM_NEXTAGE_TO_FTSENSOR_Link, child RARM_FTSENSOR_Link, origin xyz=0.0275 0.0275 -0.017 rpy=0 0 0.785398

Commit message: Update link name and refactor euslisp files

File: nextage_tutorials/urdf/JSKNextageOpen.urdf (robot description, URDF)
Before this commit: robot NextageOpen, 27 links, 26 joints
Links:
- removed link CHEST_L515_Link
- removed link CHEST_NEXTAGE_TO_L515_Link
- removed link L515_Link
- added link CHEST_NEXTAGE_TO_TOP_CAMERA_Link; collision mesh filename=package://nextage_tutorials/meshes/CHEST_NEXTAGE_TO_L515.stl scale=0.001 0.001 0.001; visual mesh filename=package://nextage_tutorials/meshes/CHEST_NEXTAGE_TO_L515.stl scale=0.001 0.001 0.001
- added link TOP_CAMERA_Link; collision mesh filename=package://nextage_tutorials/meshes/CHEST_L515.stl scale=0.001 0.001 0.001; visual mesh filename=package://nextage_tutorials/meshes/CHEST_L515.stl scale=0.001 0.001 0.001
- added link top_camera_link; collision mesh filename=package://nextage_tutorials/meshes/L515.stl scale=0.001 0.001 0.001; visual mesh filename=package://nextage_tutorials/meshes/L515.stl scale=0.001 0.001 0.001
Joints:
- removed joint CHEST_JOINT0_TO_NEXTAGE_TO_L515
- removed joint CHEST_L515_TO_L515
- removed joint CHEST_NEXTAGE_TO_L515_TO_CHEST_L515
- added joint CHEST_JOINT0_TO_NEXTAGE_TO_TOP_CAMERA: type fixed, parent CHEST_JOINT0_Link, child CHEST_NEXTAGE_TO_TOP_CAMERA_Link, origin xyz=0.080855 0.099197 0.291294 rpy=0.698132 0 -1.570796
- added joint CHEST_NEXTAGE_TO_TOP_CAMERA_TO_TOP_CAMERA: type fixed, parent CHEST_NEXTAGE_TO_TOP_CAMERA_Link, child TOP_CAMERA_Link, origin xyz=0.099197 0.069502 0.025 rpy=-1.570796 1.570796 0
- added joint TOP_CAMERA_TO_TOP_CAMERA: type fixed, parent TOP_CAMERA_Link, child top_camera_link, origin xyz=0 0 0 rpy=0 0 0

Commit message: Update camera tf

File: nextage_tutorials/urdf/JSKNextageOpen.urdf (robot description, URDF)
Before this commit: robot NextageOpen, 27 links, 26 joints
Joints:
- joint TOP_CAMERA_TO_TOP_CAMERA: origin xyz=0 0 0 rpy=0 0 0 -> xyz=0 0 0 rpy=1.570796 0 0

Commit message: Add camera frame to URDF

File: nextage_tutorials/urdf/JSKNextageOpen.urdf (robot description, URDF)
Before this commit: robot NextageOpen, 27 links, 26 joints
Links:
- added link LARM_CAMERA_Link; collision box size=0.025 0.025 0.025; visual box size=0.025 0.025 0.025
- added link RARM_CAMERA_Link; collision box size=0.025 0.025 0.025; visual box size=0.025 0.025 0.025
Joints:
- added joint LARM_CAMERA_Joint: type fixed, parent LARM_JOINT5_Link, child LARM_CAMERA_Link, origin xyz=0.02 0.045 -0.03 rpy=1.21300383 0 1.881464934
- added joint RARM_CAMERA_Joint: type fixed, parent RARM_JOINT5_Link, child RARM_CAMERA_Link, origin xyz=0.02 -0.045 -0.03 rpy=1.21300383 0 1.26012772

File: nextage_tutorials/urdf/JSKNextageOpenGripper.urdf (robot description, URDF)
Before this commit: robot JSKNextageOpenGripper, 45 links, 44 joints
Links:
- added link LARM_CAMERA_Link; collision box size=0.025 0.025 0.025; visual box size=0.025 0.025 0.025
- added link RARM_CAMERA_Link; collision box size=0.025 0.025 0.025; visual box size=0.025 0.025 0.025
Joints:
- added joint LARM_CAMERA_Joint: type fixed, parent LARM_JOINT5_Link, child LARM_CAMERA_Link, origin xyz=0.02 0.045 -0.03 rpy=1.21300383 0 1.881464934
- added joint RARM_CAMERA_Joint: type fixed, parent RARM_JOINT5_Link, child RARM_CAMERA_Link, origin xyz=0.02 -0.045 -0.03 rpy=1.21300383 0 1.26012772

Commit message: Maintain cameras and sensors

File: nextage_tutorials/urdf/JSKNextageOpen.urdf (robot description, URDF)
Before this commit: robot NextageOpen, 29 links, 28 joints
Links:
- added link LARM_FTSENSOR_SENSOR_Link
- added link RARM_FTSENSOR_SENSOR_Link
Joints:
- added joint LARM_FTSENSOR_TO_FTSENSOR_SENSOR: type fixed, parent LARM_FTSENSOR_Link, child LARM_FTSENSOR_SENSOR_Link, origin xyz=0 0 0 rpy=0 3.141593 0
- added joint RARM_FTSENSOR_TO_FTSENSOR_SENSOR: type fixed, parent RARM_FTSENSOR_Link, child RARM_FTSENSOR_SENSOR_Link, origin xyz=0 0 0 rpy=0 3.141593 0
- joint TOP_CAMERA_TO_TOP_CAMERA: origin xyz=0 0 0 rpy=1.570796 0 0 -> xyz=0 0 0 rpy=0 0 0

File: nextage_tutorials/urdf/JSKNextageOpenGripper.urdf (robot description, URDF)
Before this commit: robot JSKNextageOpenGripper, 47 links, 46 joints
Links:
- added link LARM_FTSENSOR_SENSOR_Link
- added link RARM_FTSENSOR_SENSOR_Link
- link lhand_base_link: geometry collision mesh filename=package://dynamixel_detachable_hand/meshes/nejineji_finger_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; visual mesh filename=package://dynamixel_detachable_hand/meshes/nejineji_finger_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
- link lhand_bottom_spacer3300a_1: geometry collision mesh filename=package://dynamixel_detachable_hand/meshes/nejineji_finger_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; visual mesh filename=package://dynamixel_detachable_hand/meshes/nejineji_finger_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
- link lhand_finger_11: geometry collision mesh filename=package://dynamixel_detachable_hand/meshes/nejineji_finger_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; visual mesh filename=package://dynamixel_detachable_hand/meshes/nejineji_finger_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
- link lhand_finger_13: geometry collision mesh filename=package://dynamixel_detachable_hand/meshes/nejineji_finger_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; visual mesh filename=package://dynamixel_detachable_hand/meshes/nejineji_finger_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
- link lhand_pinion_1: geometry collision mesh filename=package://dynamixel_detachable_hand/meshes/nejineji_finger_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; visual mesh filename=package://dynamixel_detachable_hand/meshes/nejineji_finger_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
- link lhand_screwlock_male_1: geometry collision mesh filename=package://dynamixel_detachable_hand/meshes/nejineji_finger_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; visual mesh filename=package://dynamixel_detachable_hand/meshes/nejineji_finger_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
- link lhand_small_diameter_hornb_1: geometry collision mesh filename=package://dynamixel_detachable_hand/meshes/nejineji_finger_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; visual mesh filename=package://dynamixel_detachable_hand/meshes/nejineji_finger_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
- link lhand_xl_xc_330_1_2: geometry collision mesh filename=package://dynamixel_detachable_hand/meshes/nejineji_finger_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; visual mesh filename=package://dynamixel_detachable_hand/meshes/nejineji_finger_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
- link rhand_base_link: geometry collision mesh filename=package://dynamixel_detachable_hand/meshes/nejineji_finger_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; visual mesh filename=package://dynamixel_detachable_hand/meshes/nejineji_finger_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
- link rhand_bottom_spacer3300a_1: geometry collision mesh filename=package://dynamixel_detachable_hand/meshes/nejineji_finger_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; visual mesh filename=package://dynamixel_detachable_hand/meshes/nejineji_finger_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
- link rhand_finger_11: geometry collision mesh filename=package://dynamixel_detachable_hand/meshes/nejineji_finger_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; visual mesh filename=package://dynamixel_detachable_hand/meshes/nejineji_finger_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
- link rhand_finger_13: geometry collision mesh filename=package://dynamixel_detachable_hand/meshes/nejineji_finger_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; visual mesh filename=package://dynamixel_detachable_hand/meshes/nejineji_finger_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
- link rhand_pinion_1: geometry collision mesh filename=package://dynamixel_detachable_hand/meshes/nejineji_finger_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; visual mesh filename=package://dynamixel_detachable_hand/meshes/nejineji_finger_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
- link rhand_screwlock_male_1: geometry collision mesh filename=package://dynamixel_detachable_hand/meshes/nejineji_finger_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; visual mesh filename=package://dynamixel_detachable_hand/meshes/nejineji_finger_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
- link rhand_small_diameter_hornb_1: geometry collision mesh filename=package://dynamixel_detachable_hand/meshes/nejineji_finger_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; visual mesh filename=package://dynamixel_detachable_hand/meshes/nejineji_finger_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
- link rhand_xl_xc_330_1_2: geometry collision mesh filename=package://dynamixel_detachable_hand/meshes/nejineji_finger_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; visual mesh filename=package://dynamixel_detachable_hand/meshes/nejineji_finger_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
Joints:
- added joint LARM_FTSENSOR_TO_FTSENSOR_SENSOR: type fixed, parent LARM_FTSENSOR_Link, child LARM_FTSENSOR_SENSOR_Link, origin xyz=0 0 0 rpy=0 3.141593 0
- added joint RARM_FTSENSOR_TO_FTSENSOR_SENSOR: type fixed, parent RARM_FTSENSOR_Link, child RARM_FTSENSOR_SENSOR_Link, origin xyz=0 0 0 rpy=0 3.141593 0
- joint TOP_CAMERA_TO_TOP_CAMERA: origin xyz=0 0 0 rpy=1.570796 0 0 -> xyz=0 0 0 rpy=0 0 0

Commit message: Update d405 frame

File: nextage_tutorials/urdf/JSKNextageOpen.urdf (robot description, URDF)
Before this commit: robot NextageOpen, 31 links, 30 joints
Joints:
- joint RARM_CAMERA_Joint: origin xyz=0.02 -0.045 -0.03 rpy=1.21300383 0 1.26012772 -> xyz=-0.0762682557 0.0627098233 -0.0274769068 rpy=1.81198951 -0.00861059949 -2.60779872

File: nextage_tutorials/urdf/JSKNextageOpenGripper.urdf (robot description, URDF)
Before this commit: robot JSKNextageOpenGripper, 49 links, 48 joints
Joints:
- joint RARM_CAMERA_Joint: origin xyz=0.02 -0.045 -0.03 rpy=1.21300383 0 1.26012772 -> xyz=-0.0762682557 0.0627098233 -0.0274769068 rpy=1.81198951 -0.00861059949 -2.60779872
